File: vusb_version.brd (EAGLE design)
At the start: 28.9 x 40.6 mm, 25 parts

Commit message: printed version 2
debugged, optimized, working, woots.
Parts:
- moved R1 5.39 mm to (75.6, 40.0), turned to 0 degrees
- moved D2 4.45 mm to (76.2, 45.7), turned to 270 degrees
- moved R2 3.17 mm to (75.6, 42.5)
- moved R3 1.91 mm to (79.4, 40.0)
- moved D1 0.63 mm to (81.9, 45.1)
- moved JP1 0.32 mm to (80.3, 52.1)
Routing:
- net USBD-: track 9.84 -> 4.32 mm
- net VCC: track 39.3 -> 36.6 mm
- net USBD+: track 3.59 -> 6.20 mm
- net GND: track 13.0 -> 11.1 mm
- net D-: track 13.6 -> 12.3 mm
Other:
- board size 28.9 x 40.6 mm -> 29.2 x 40.6 mm
