File: megaUSB_spider.sch (EAGLE design)
At the start: 23 parts

Commit message: cleanup of the old versions
Parts:
- added RIGHT-SIDE, SERIAL: (no value), pinhead:PINHD-1X3
Connections:
- net GND: now also RIGHT-SIDE.1, SERIAL.3; no longer PROG.2, RESET.2
- net PD0: now also SERIAL.1
- net PD1: now also SERIAL.2
- net PROG: now also ATMEGAX8.5; no longer ATMEGAX8.6, PROG.3
- net RESET: no longer RESET.4
- net USBD-: now also ATMEGAX8.6; no longer ATMEGAX8.5
- net VCC: now also RIGHT-SIDE.3
Changed lines of the file:
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@@
 <part name="R8" library="SparkFun-Passives" deviceset="RESISTOR" device="1206" value="220 ohm"/>
 <part name="Y2" library="SparkFun-FreqCtrl" deviceset="CRYSTAL" device="HC49US"/>
+<part name="RIGHT-SIDE" library="pinhead" deviceset="PINHD-1X3" device=""/>
+<part name="SERIAL" library="pinhead" deviceset="PINHD-1X3" device=""/>
 </parts>
 <sheets>
@@
 <instance part="R8" gate="G$1" x="154.94" y="27.94" rot="R90"/>
 <instance part="Y2" gate="G$1" x="53.34" y="53.34"/>
+<instance part="RIGHT-SIDE" gate="A" x="127" y="76.2"/>
+<instance part="SERIAL" gate="A" x="71.12" y="73.66"/>
 </instances>
 <busses>
@@
 </segment>
 <segment>
-<pinref part="RESET" gate="S" pin="4"/>
 <pinref part="RESET" gate="S" pin="3"/>
-<wire x1="20.32" y1="53.34" x2="20.32" y2="55.88" width="0.1524" layer="91"/>
 <wire x1="20.32" y1="55.88" x2="27.94" y2="55.88" width="0.1524" layer="91"/>
-<junction x="20.32" y="55.88"/>
 <label x="27.94" y="55.88" size="1.778" layer="95"/>
 </segment>
@@
 <label x="78.74" y="76.2" size="1.778" layer="95"/>
 </segment>
+<segment>
+<pinref part="SERIAL" gate="A" pin="1"/>
+<wire x1="68.58" y1="76.2" x2="55.88" y2="76.2" width="0.1524" layer="91"/>
+<label x="55.88" y="76.2" size="1.778" layer="95"/>
+</segment>
 </net>
 <net name="PD1" class="0">
@@
 <wire x1="91.44" y1="73.66" x2="78.74" y2="73.66" width="0.1524" layer="91"/>
 <label x="78.74" y="73.66" size="1.778" layer="95"/>
+</segment>
+<segment>
+<pinref part="SERIAL" gate="A" pin="2"/>
+<wire x1="68.58" y1="73.66" x2="55.88" y2="73.66" width="0.1524" layer="91"/>
+<label x="55.88" y="73.66" size="1.778" layer="95"/>
 </segment>
 </net>
@@
 <pinref part="SUPPLY9" gate="G$1" pin="VCC"/>
 </segment>
+<segment>
+<pinref part="RIGHT-SIDE" gate="A" pin="3"/>
+<wire x1="124.46" y1="73.66" x2="109.22" y2="73.66" width="0.1524" layer="91"/>
+<label x="109.22" y="73.66" size="1.778" layer="95"/>
+</segment>
 </net>
 <net name="GND" class="0">
@@
 <segment>
 <pinref part="RESET" gate="S" pin="1"/>
-<pinref part="RESET" gate="S" pin="2"/>
 <wire x1="2.54" y1="55.88" x2="10.16" y2="55.88" width="0.1524" layer="91"/>
-<wire x1="10.16" y1="55.88" x2="10.16" y2="53.34" width="0.1524" layer="91"/>
 <label x="2.54" y="55.88" size="1.778" layer="95"/>
 </segment>
 <segment>
 <pinref part="PROG" gate="S" pin="1"/>
-<pinref part="PROG" gate="S" pin="2"/>
 <wire x1="2.54" y1="38.1" x2="10.16" y2="38.1" width="0.1524" layer="91"/>
-<wire x1="10.16" y1="38.1" x2="10.16" y2="35.56" width="0.1524" layer="91"/>
 <label x="2.54" y="38.1" size="1.778" layer="95"/>
 </segment>
@@
 <pinref part="SUPPLY12" gate="GND" pin="GND"/>
 <wire x1="154.94" y1="22.86" x2="154.94" y2="20.32" width="0.1524" layer="91"/>
+</segment>
+<segment>
+<pinref part="RIGHT-SIDE" gate="A" pin="1"/>
+<wire x1="124.46" y1="78.74" x2="109.22" y2="78.74" width="0.1524" layer="91"/>
+<label x="109.22" y="78.74" size="1.778" layer="95"/>
+</segment>
+<segment>
+<pinref part="SERIAL" gate="A" pin="3"/>
+<wire x1="68.58" y1="71.12" x2="55.88" y2="71.12" width="0.1524" layer="91"/>
+<label x="55.88" y="71.12" size="1.778" layer="95"/>
 </segment>
 </net>
@@
 <net name="PROG" class="0">
 <segment>
+<label x="27.94" y="38.1" size="1.778" layer="95"/>
 <pinref part="PROG" gate="S" pin="4"/>
-<pinref part="PROG" gate="S" pin="3"/>
-<wire x1="20.32" y1="35.56" x2="20.32" y2="38.1" width="0.1524" layer="91"/>
-<wire x1="20.32" y1="38.1" x2="27.94" y2="38.1" width="0.1524" layer="91"/>
-<junction x="20.32" y="38.1"/>
-<label x="27.94" y="38.1" size="1.778" layer="95"/>
-</segment>
-<segment>
-<pinref part="ATMEGAX8" gate="A" pin="6"/>
-<wire x1="91.44" y1="66.04" x2="78.74" y2="66.04" width="0.1524" layer="91"/>
-<label x="78.74" y="66.04" size="1.778" layer="95"/>
+<wire x1="20.32" y1="35.56" x2="27.94" y2="35.56" width="0.1524" layer="91"/>
+<wire x1="27.94" y1="35.56" x2="27.94" y2="38.1" width="0.1524" layer="91"/>
+</segment>
+<segment>
+<pinref part="ATMEGAX8" gate="A" pin="5"/>
+<wire x1="91.44" y1="68.58" x2="78.74" y2="68.58" width="0.1524" layer="91"/>
+<label x="78.74" y="68.58" size="1.778" layer="95"/>
 </segment>
 </net>
@@
 </segment>
 <segment>
-<pinref part="ATMEGAX8" gate="A" pin="5"/>
-<wire x1="91.44" y1="68.58" x2="78.74" y2="68.58" width="0.1524" layer="91"/>
-<label x="78.74" y="68.58" size="1.778" layer="95"/>
-</segment>
-</net>
+<pinref part="ATMEGAX8" gate="A" pin="6"/>
+<wire x1="91.44" y1="66.04" x2="78.74" y2="66.04" width="0.1524" layer="91"/>
+<label x="78.74" y="66.04" size="1.778" layer="95"/>
+</segment>
+</net>
